File: v3/CM5_GPIO.kicad_sch (KiCad schematic)
At the start: 29 parts, among them J4 Conn_01x02, J5 UART Connection, J6 Micro_SD_Card_Det, Q1 AO3400A, SW1 Right angle Tact button, SW2 Right angle Tact button, U1 74LVC1G07SE-7, U2 ASM330LHHTR, U3 XIAO_RM3100_Breakout, U4 RT9742GGJ5, U5 LSM9DS1

Commit message: Various pcb mods
Parts:
- removed Module1: ComputeModule5-CM5, CM5IO:Raspberry-Pi-5-Compute-Module, symbol CM5IO:ComputeModule5-CM5
- added J9: 10164227-1001A1RLF, CM5IO:CM5_connector, symbol cm5_a:CM5_a
- C10: renamed from C5; LCSC PN (none) -> C117956
- C11: renamed from C6; LCSC PN (none) -> C117956
- C3: renamed from C11; Field6 (none) -> RM EMK105 B7103KV-F; Field7 (none) -> TAIYO YUDEN EUROPE GMBH; LCSC PN (none) -> C414271
- C4: renamed from C10; LCSC PN (none) -> C92753
- C5: renamed from C9; LCSC PN (none) -> C92753
- C6: renamed from C8; LCSC PN (none) -> C117956
- C7: LCSC PN (none) -> C92753
- C8: renamed from C3; LCSC PN (none) -> C92753
- C9: renamed from C4; LCSC PN (none) -> C92753
- D1: LCSC PN (none) -> C273616
- D2: LCSC PN (none) -> C19171323
- J5: renamed from J4; Field6 (none) -> JST_PH_S2B-PH-SM4-TB; LCSC PN (none) -> C295747
- J6: renamed from J5; Field5 (none) -> nf; Field6 (none) -> nf; Field7 (none) -> nf
- J7: renamed from J6; LCSC PN (none) -> C428492
- LS1: value AST1240MLTRQ -> KMTG1203; Field6 (none) -> KMTG1203; LCSC PN (none) -> C7421651
- Q1: Field6 (none) -> AO3400A; LCSC PN (none) -> C20917
- R5, R6: Field6 RK73H1ETTP1001F -> 0402WGF1001TCE; LCSC PN (none) -> C11702
- R7: Field6 (none) -> 0402WGF1800TCE; LCSC PN (none) -> C38941; Part Description Resistor 2.2K M1005 1% 63mW -> Resistor 180 M1005 1% 63mW
- R8, R9: Field6 (none) -> 0402WGF2201TCE; LCSC PN (none) -> C25879
- SW1, SW2: LCSC PN (none) -> C221888
- U1: renamed from U5; Field6 (none) -> LSM9DS1; LCSC PN (none) -> C2655096
- U2: renamed from U1; LCSC PN (none) -> C67531
- U3: renamed from U2; Field6 (none) -> ASM330LHHTR; LCSC PN (none) -> C459826
- U4: renamed from U3; Field5 (none) -> nf; Field6 (none) -> nf; Field7 (none) -> nf
- U5: renamed from U4; LCSC PN (none) -> C250547
Connections:
- net +1.8v: now also J9.88 (+1.8v_(Output)), J9.90 (+1.8v_(Output))
- net +3.3v: now also J9.78 (GPIO_VREF(1.8v/3.3v_Input)), J9.84 (+3.3v_(Output)), J9.86 (+3.3v_(Output))
- net +5v: now also J9.77 (+5v_(Input)), J9.79 (+5v_(Input)), J9.81 (+5v_(Input)), J9.83 (+5v_(Input)), J9.85 (+5v_(Input)), J9.87 (+5v_(Input))
- net BT_nDis: now also J9.91 (BT_nDisable)
- net CAM_GPIO0: now also J9.97 (CAM_GPIO0)
- net CAM_GPIO1: now also J9.100 (CAM_GPIO1)
- net CC1: now also J9.94 (CC1)
- net CC2: now also J9.96 (CC2)
- net EEPROM_nWP: now also J9.20 (EEPROM_nWP)
- net ETH_LEDG: now also J9.17 (Ethernet_nLED2(3.3v))
- net ETH_LEDY: now also J9.15 (Ethernet_nLED3(3.3v))
- net GND: now also J9.1 (GND), J9.13 (GND), J9.14 (GND), J9.2 (GND), J9.22 (GND), J9.23 (GND), J9.32 (GND), J9.33 (GND), J9.42 (GND), J9.43 (GND), J9.52 (GND), J9.53 (GND), J9.59 (GND), J9.60 (GND), J9.65 (GND), J9.66 (GND), J9.7 (GND), J9.71 (GND), J9.74 (GND), J9.8 (GND), J9.98 (GND)
- net GPIO10: now also J9.44 (GPIO10)
- net GPIO11: now also J9.38 (GPIO11)
- net GPIO12: now also J9.31 (GPIO12)
- net GPIO13: now also J9.28 (GPIO13)
- net GPIO14: now also J9.55 (GPIO14)
- net GPIO15: now also J9.51 (GPIO15)
- net GPIO16: now also J9.29 (GPIO16)
- net GPIO17: now also J9.50 (GPIO17)
- net GPIO18: now also J9.49 (GPIO18)
- net GPIO19: now also J9.26 (GPIO19)
- net GPIO2: now also J9.58 (GPIO2)
- net GPIO20: now also J9.27 (GPIO20)
- net GPIO21: now also J9.25 (GPIO21)
- net GPIO22: now also J9.46 (GPIO22)
- net GPIO23: now also J9.47 (GPIO23)
- net GPIO24: now also J9.45 (GPIO24)
- net GPIO25: now also J9.41 (GPIO25)
- net GPIO26: now also J9.24 (GPIO26)
- net GPIO27: now also J9.48 (GPIO27)
- net GPIO3: now also J9.56 (GPIO3)
- net GPIO4: now also J9.54 (GPIO4)
- net GPIO5: now also J9.34 (GPIO5)
- net GPIO6: now also J9.30 (GPIO6)
- net GPIO7: now also J9.37 (GPIO7)
- net GPIO8: now also J9.39 (GPIO8)
- net GPIO9: now also J9.40 (GPIO9)
- net ID_SC: now also J9.35 (ID_SC)
- net ID_SD: now also J9.36 (ID_SD)
- net PMIC_ENABLE: now also J9.99 (PMIC_ENABLE)
- net PWM: now also J9.19 (FAN_PWM)
- net PWR_BUT: now also J9.92 (PWR_BUT)
- net SCL0: now also J9.80 (SCL0)
- net SDA0: now also J9.82 (SDA0)
- net SD_CLK: now also J9.57 (SD_CLK)
- net SD_CMD: now also J9.62 (SD_CMD)
- net SD_DAT0: now also J9.63 (SD_DAT0)
- net SD_DAT1: now also J9.67 (SD_DAT1)
- net SD_DAT2: now also J9.69 (SD_DAT2)
- net SD_DAT3: now also J9.61 (SD_DAT3)
- net SD_PWR_ON: now also J9.75 (SD_PWR_ON)
- net SYNC_OUT: now also J9.18 (Ethernet_SYNC_OUT(3.3v))
- net TACHO: now also J9.16 (FAN_TACHO)
- net TRD0_N: now also J9.10 (Ethernet_Pair0_N)
- net TRD0_P: now also J9.12 (Ethernet_Pair0_P)
- net TRD1_N: now also J9.6 (Ethernet_Pair1_N)
- net TRD1_P: now also J9.4 (Ethernet_Pair1_P)
- net TRD2_N: now also J9.9 (Ethernet_Pair2_N)
- net TRD2_P: now also J9.11 (Ethernet_Pair2_P)
- net TRD3_N: now also J9.5 (Ethernet_Pair3_N)
- net TRD3_P: now also J9.3 (Ethernet_Pair3_P)
- net VBAT: now also J9.76 (VBAT)
- net WL_nDis: now also J9.89 (WiFi_nDisable)
- net nPWR_LED: now also J9.95 (LED_nPWR)
- net nRPIBOOT: now also J9.93 (nRPIBOOT)
- net at R5.2: now also J9.21 (LED_nACT)

Commit message: convert to CS20 TOF
Parts:
- removed J5: Conn_01x02, Connector_JST:JST_PH_S2B-PH-SM4-TB_1x02-1MP_P2.00mm_Horizontal, symbol Connector_Generic:Conn_01x02
- removed J6: UART Connection, Connector_PinHeader_2.54mm:PinHeader_1x03_P2.54mm_Vertical, symbol Connector_Generic:Conn_01x03
- removed Q1: AO3400A, Package_TO_SOT_SMD:SOT-23, symbol Transistor_FET:AO3400A
- removed U1: LSM9DS1, Package_LGA:LGA-24L_3x3.5mm_P0.43mm, symbol Sensor_Motion:LSM9DS1
- removed U3: ASM330LHHTR, CM5IO:ASM330LHHTR, symbol ASM330LHHTR:ASM330LHHTR
- removed U4: XIAO_RM3100_Breakout, CM5IO:RM3100_Breakout, symbol STIC-rescue:RM3100_Breakout-XIAO
- added L1: XFL4020-152MEC, footprint:IND-SMD_L4.0-W4.0-A, symbol Device:L
- added R10, R11: 2.2K 1%, Resistor_SMD:R_0402_1005Metric, symbol Device:R
- added U1: TPS63020DSJR, footprint:VSON-14_L4.0-W3.0-P0.50-BL-EP_TI_DSJ, symbol TPS63020DSJR:TPS63020DSJR
- added U3: ICM-20948, CM5IO:QFN40P300X300X105-24N, symbol ICM-20948:ICM-20948
- C10: value 10u -> 100nF; footprint Capacitor_SMD:C_0805_2012Metric -> Capacitor_SMD:C_0603_1608Metric; Field4 Digikey -> (none); Field5 490-14381-1-ND -> (none); Field6 GRM21BR71A106KA73L -> (none); Field7 Murata -> (none); Field8 111893011 -> (none); LCSC (none) -> C45000; LCSC PN C117956 -> (none); Part Description 10uF 10% 10V Ceramic Capacitor X7R 0805 (2012 Metric) -> (none)
- C3: value 10n -> 100nF; footprint Capacitor_SMD:C_0402_1005Metric -> Capacitor_SMD:C_0603_1608Metric; Field6 RM EMK105 B7103KV-F -> (none); Field7 TAIYO YUDEN EUROPE GMBH -> (none); LCSC (none) -> C45000; LCSC PN C414271 -> (none)
- C4, C5, C7: value 100n -> 22uF; footprint Capacitor_SMD:C_0402_1005Metric -> Capacitor_SMD:C_1206_3216Metric; Field4 Farnell -> (none); Field5 2611911 -> (none); Field6 RM EMK105 B7104KV-F -> (none); Field7 TAIYO YUDEN EUROPE GMBH -> (none); Field8 110091611 -> (none); LCSC (none) -> C5252682; LCSC PN C92753 -> (none); Part Description 0.1uF 10% 16V Ceramic Capacitor X7R 0402 (1005 Metric) -> (none)
- C6: value 10u -> 22uF; footprint Capacitor_SMD:C_0805_2012Metric -> Capacitor_SMD:C_1206_3216Metric; Field4 Digikey -> (none); Field5 490-14381-1-ND -> (none); Field6 GRM21BR71A106KA73L -> (none); Field7 Murata -> (none); Field8 111893011 -> (none); LCSC (none) -> C5252682; LCSC PN C117956 -> (none); Part Description 10uF 10% 10V Ceramic Capacitor X7R 0805 (2012 Metric) -> (none)
- C8, C9: value 100n -> 100nF; footprint Capacitor_SMD:C_0402_1005Metric -> Capacitor_SMD:C_0603_1608Metric; Field4 Farnell -> (none); Field5 2611911 -> (none); Field6 RM EMK105 B7104KV-F -> (none); Field7 TAIYO YUDEN EUROPE GMBH -> (none); Field8 110091611 -> (none); LCSC (none) -> C45000; LCSC PN C92753 -> (none); Part Description 0.1uF 10% 16V Ceramic Capacitor X7R 0402 (1005 Metric) -> (none)
- R8: value 2.2K 1% -> 1M; footprint Resistor_SMD:R_0402_1005Metric -> Resistor_SMD:R_0603_1608Metric; Field4 Farnell -> (none); Field6 0402WGF2201TCE -> (none); LCSC (none) -> C227459; LCSC PN C25879 -> (none); Part Description Resistor 2.2K M1005 1% 63mW -> (none)
- R9: value 2.2K 1% -> 180k; footprint Resistor_SMD:R_0402_1005Metric -> Resistor_SMD:R_0603_1608Metric; Field4 Farnell -> (none); Field6 0402WGF2201TCE -> (none); LCSC (none) -> C227451; LCSC PN C25879 -> (none); Part Description Resistor 2.2K M1005 1% 63mW -> (none)
Connections:
- net +1.8v: now also C10.1, C9.1, J9.78 (GPIO_VREF(1.8v/3.3v_Input)), R10.1, R11.1, U3.13 (VDD), U3.22 (~{CS}), U3.8 (VDDIO)
- net +3.3v: no longer C10.1, C5.1, C6.1, C7.1, C8.1, C9.1, J9.78 (GPIO_VREF(1.8v/3.3v_Input)), R8.1, R9.1
- net GND: now also C3.1, R9.1, U1.15 (PGND), U1.2 (GND), U3.18 (GND), U3.20 (RESV_20), U3.9 (AD0/SDO); no longer C3.2
- net GPIO14: now also R11.2, U3.24 (SDA/SDI)
- net GPIO15: now also R10.2, U3.23 (SCL/SCLK)
- net GPIO2: no longer R8.2
- net GPIO23: now also U3.11 (FSYNC)
- net GPIO24: now also U3.12 (INT1)
- net GPIO27: now also U1.14 (PG)
- net GPIO3: no longer R9.2
- net +3.3vLED: now reaches C4.1
- net +3.3vLED: now also C5.1, C6.1, R8.1, U1.4 (VOUT), U1.5 (VOUT)
- net GPIO22 renamed EN
- net EN: now also U1.12 (EN)
- net GPIO5 renamed CAM_CLK
- net GPIO6 renamed CAM_RST
- new net: R8.2, R9.2, U1.3 (FB)
- new net: C8.1, U3.10 (REGOUT)
- new net: C3.2, U1.1 (VINA)
- new net: L1.1, U1.6 (L2), U1.7 (L2)
- new net: L1.2, U1.8 (L1), U1.9 (L1)
- new net: U3.1 (NC), U3.14 (NC), U3.15 (NC), U3.16 (NC), U3.17 (NC), U3.2 (NC), U3.3 (NC), U3.4 (NC), U3.5 (NC), U3.6 (NC)
- new net +5V: C7.1, U1.10 (VIN), U1.11 (VIN), U1.13 (PS/SYNC)
- no-connect marks 8 -> 9
