File: v3/CM5_GPIO.kicad_sch (KiCad schematic)
At the start: 29 parts, among them J5 Conn_01x02, J6 UART Connection, J7 Micro_SD_Card_Det, J9 10164227-1001A1RLF, Q1 AO3400A, SW1 Right angle Tact button, SW2 Right angle Tact button, U1 LSM9DS1, U2 74LVC1G07SE-7, U3 ASM330LHHTR, U4 XIAO_RM3100_Breakout, U5 RT9742GGJ5

Commit message: adding power management to board
Parts:
- removed C10, C6: 10u, Capacitor_SMD:C_0805_2012Metric, symbol Device:C
- removed C3: 10n, Capacitor_SMD:C_0402_1005Metric, symbol Device:C
- removed C4, C5, C7, C8, C9: 100n, Capacitor_SMD:C_0402_1005Metric, symbol Device:C
- removed J5: Conn_01x02, Connector_JST:JST_PH_S2B-PH-SM4-TB_1x02-1MP_P2.00mm_Horizontal, symbol Connector_Generic:Conn_01x02
- removed Q1: AO3400A, Package_TO_SOT_SMD:SOT-23, symbol Transistor_FET:AO3400A
- removed R8, R9: 2.2K 1%, Resistor_SMD:R_0402_1005Metric, symbol Device:R
- removed SW1: Right angle Tact button, Button_Switch_THT:SW_Tactile_SPST_Angled_PTS645Vx58-2LFS, symbol Switch:SW_Push
- removed U1: LSM9DS1, Package_LGA:LGA-24L_3x3.5mm_P0.43mm, symbol Sensor_Motion:LSM9DS1
- removed U3: ASM330LHHTR, CM5IO:ASM330LHHTR, symbol ASM330LHHTR:ASM330LHHTR
- removed U4: XIAO_RM3100_Breakout, CM5IO:RM3100_Breakout, symbol STIC-rescue:RM3100_Breakout-XIAO
- added J4: Conn_01x04_Pin, Connector_FFC-FPC:JUSHUO_AFA07-S04FCA-00_1x4-1MP_P1.0mm_Horizontal, symbol Connector:Conn_01x04_Pin
- C11: value 10u -> 10uF
Connections:
- net GND: now also J4.1 (Pin_1)
- net GPIO2 renamed PWR_SDA
- net GPIO3 renamed PWR_SCL
- new net +3V3: J4.4 (Pin_4)
- new net SCL3V3: J4.3 (Pin_3)
- new net SDA3V3: J4.2 (Pin_2)

Commit message: Finalise v1.0 design
Parts:
- removed D1: LED Green, LED_SMD:LED_0603_1608Metric, symbol Device:LED
- removed D2: LED Red, LED_SMD:LED_0603_1608Metric, symbol Device:LED
- removed SW2: Right angle Tact button, Button_Switch_THT:SW_Tactile_SPST_Angled_PTS645Vx58-2LFS, symbol Switch:SW_Push
- added LED1: MHS171CYCT, footprint:LED-SMD_L2.0-W1.1-R-RD-SIDE_YELLOW, symbol MHS171CYCT:MHS171CYCT
- added LED2: MHS171UGCT, footprint:LED-SMD_L2.0-W1.1_RD_GREEN_SIDE, symbol MHS171UGCT:MHS171UGCT
- added R2, R20, R21, R3: 2.2K 1%, Resistor_SMD:R_0402_1005Metric, symbol Device:R
- added SW1: TS-1093C-A14B3-D1, footprint:SW-TH_TS-1093C-A14B3-D1, symbol TS-1093C-A14B3-D1:TS-1093C-A14B3-D1
- J5: renamed from J4; LCSC PN (none) -> C262710
- renumbered C11 to C1, J9 to J6, J6 to J8, R7 to R6, R6 to R7, U2 to U3, U5 to U4
Connections:
- net +3V3 is gone; now on net +3.3v: J5.4 (Pin_4)
- net SCL3V3 is gone; now on net PWR_SCL: J5.3 (Pin_3)
- net SDA3V3 is gone; now on net PWR_SDA: J5.2 (Pin_2)
- net +3.3v: now also LED1.1 (K), LED2.1 (+), R2.1, R20.1, R21.1, R3.1
- net GND: now also SW1.1
- net ID_SC: now also R3.2
- net ID_SD: now also R2.2
- net PWR_SCL: now also R20.2
- net PWR_SDA: now also R21.2
- net at R5.1: now also LED1.2 (A)
- net at R7.1: now also LED2.2 (-)
- net BT_nDis: no longer names the net of J6.91 (BT_nDisable)
- net CC1: no longer names the net of J6.94 (CC1)
- net CC2: no longer names the net of J6.96 (CC2)
- net EEPROM_nWP: no longer names the net of J6.20 (EEPROM_nWP)
- net ETH_LEDG: no longer names the net of J6.17 (Ethernet_nLED2(3.3v))
- net ETH_LEDY: no longer names the net of J6.15 (Ethernet_nLED3(3.3v))
- net GPIO10: no longer names the net of J6.44 (GPIO10)
- net GPIO11: no longer names the net of J6.38 (GPIO11)
- net GPIO12 renamed BUZZ_B
- net BUZZ_B: now also LS1.2
- net GPIO13: no longer names the net of J6.28 (GPIO13)
- net GPIO13: no longer LS1.2
- net GPIO16: no longer names the net of J6.29 (GPIO16)
- net GPIO17: no longer names the net of J6.50 (GPIO17)
- net GPIO18 renamed BUZZ_A
- net BUZZ_A: now also R6.1
- net GPIO19: no longer names the net of J6.26 (GPIO19)
- net GPIO19: no longer R6.1
- net GPIO20 renamed BUTTON
- net BUTTON: now also SW1.2
- net GPIO21: no longer names the net of J6.25 (GPIO21)
- net GPIO22: no longer names the net of J6.46 (GPIO22)
- net GPIO23: no longer names the net of J6.47 (GPIO23)
- net GPIO24: no longer names the net of J6.45 (GPIO24)
- net GPIO25: no longer names the net of J6.41 (GPIO25)
- net GPIO26: no longer names the net of J6.24 (GPIO26)
- net GPIO27: no longer names the net of J6.48 (GPIO27)
- net GPIO4: no longer names the net of J6.54 (GPIO4)
- net GPIO5: no longer names the net of J6.34 (GPIO5)
- net GPIO6: no longer names the net of J6.30 (GPIO6)
- net GPIO7: no longer names the net of J6.37 (GPIO7)
- net GPIO8: no longer names the net of J6.39 (GPIO8)
- net GPIO9: no longer names the net of J6.40 (GPIO9)
- net PMIC_ENABLE: no longer names the net of J6.99 (PMIC_ENABLE)
- net PWM: no longer names the net of J6.19 (FAN_PWM)
- net SYNC_OUT: no longer names the net of J6.18 (Ethernet_SYNC_OUT(3.3v))
- net TACHO: no longer names the net of J6.16 (FAN_TACHO)
- net TRD0_N: no longer names the net of J6.10 (Ethernet_Pair0_N)
- net TRD0_P: no longer names the net of J6.12 (Ethernet_Pair0_P)
- net TRD1_N: no longer names the net of J6.6 (Ethernet_Pair1_N)
- net TRD1_P: no longer names the net of J6.4 (Ethernet_Pair1_P)
- net TRD2_N: no longer names the net of J6.9 (Ethernet_Pair2_N)
- net TRD2_P: no longer names the net of J6.11 (Ethernet_Pair2_P)
- net TRD3_N: no longer names the net of J6.5 (Ethernet_Pair3_N)
- net TRD3_P: no longer names the net of J6.3 (Ethernet_Pair3_P)
- net VBAT: no longer names the net of J6.76 (VBAT)
- net WL_nDis: no longer names the net of J6.89 (WiFi_nDisable)
- net nRPIBOOT: no longer names the net of J6.93 (nRPIBOOT)
- no-connect marks 8 -> 50
Other:
- moved on the sheet: J8
