File: v3/CM5_HighSpeed.kicad_sch (KiCad schematic)
At the start: 6 parts, among them J2 Conn_01x22_Female, J3 Conn_01x22_Female, J8 10164227-1001A1RLF

Commit message: Finalise v1.0 design
Parts:
- removed J2, J3: Conn_01x22_Female, CM5IO:Hirose_FH12-22S-0.5SH_1x22-1MP_P0.50mm_Horizontal, symbol Connector:Conn_01x22_Socket
- removed R3, R4: 2.2K 1%, Resistor_SMD:R_0402_1005Metric, symbol Device:R
- added P1: AFC07-S22FCC-00 (Bottom contact), footprint:FPC-SMD_AFC07-S22FCC-00, symbol FPC_0_5MM_22P_Pull_type_H2_0mm_Under_the_next:FPC_0_5MM_22P_Pull_type_H2_0mm_Un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
- added P3: FPC_0_5MM_22P_Pull_type_H2_0mm_Pick_up, footprint:FPC-SMD_P0.50-22P_LSSJ-H2.0-22P, symbol FPC_0_5MM_22P_Pull_type_H2_0mm_Pick_up:FPC_0_5MM_22P_Pull_type_H2_0mm_Pick_up
- renumbered J8 to J3, R2 to R4
Connections:
- net +3.3v: now also P1.1, P3.1
- net CAM_GPIO0: now also P3.6
- net CAM_GPIO1: now also P3.5
- net DPHY0_C_N: now also P3.15
- net DPHY0_C_P: now also P3.14
- net DPHY0_D0_N: now also P3.21
- net DPHY0_D0_P: now also P3.20
- net DPHY0_D1_N: now also P3.18
- net DPHY0_D1_P: now also P3.17
- net DPHY0_D2_N: now also P3.12
- net DPHY0_D2_P: now also P3.11
- net DPHY0_D3_N: now also P3.9
- net DPHY0_D3_P: now also P3.8
- net DPHY1_C_N: now also P1.15
- net DPHY1_C_P: now also P1.14
- net DPHY1_D0_N: now also P1.21
- net DPHY1_D0_P: now also P1.20
- net DPHY1_D1_N: now also P1.18
- net DPHY1_D1_P: now also P1.17
- net DPHY1_D2_N: now also P1.12
- net DPHY1_D2_P: now also P1.11
- net DPHY1_D3_N: now also P1.9
- net DPHY1_D3_P: now also P1.8
- net GND: now also P1.10, P1.13, P1.16, P1.19, P1.22, P1.4, P1.7, P3.10, P3.13, P3.16, P3.19, P3.22, P3.4, P3.7
- net ID_SC: now also P1.3
- net ID_SD: now also P1.2
- net SCL0: now also P3.3
- net SDA0: now also P3.2
- net at R4.2: now also P1.6
- net HDMI0_CEC: no longer names the net of J3.51 (HDMI0_CEC)
- net HDMI0_CK_N: no longer names the net of J3.90 (HDMI0_CLK_N)
- net HDMI0_CK_P: no longer names the net of J3.88 (HDMI0_CLK_P)
- net HDMI0_D0_N: no longer names the net of J3.84 (HDMI0_TX0_N)
- net HDMI0_D0_P: no longer names the net of J3.82 (HDMI0_TX0_P)
- net HDMI0_D1_N: no longer names the net of J3.78 (HDMI0_TX1_N)
- net HDMI0_D1_P: no longer names the net of J3.76 (HDMI0_TX1_P)
- net HDMI0_D2_N: no longer names the net of J3.72 (HDMI0_TX2_N)
- net HDMI0_D2_P: no longer names the net of J3.70 (HDMI0_TX2_P)
- net HDMI0_HOTPLUG: no longer names the net of J3.53 (HDMI0_HOTPLUG)
- net HDMI0_SCL: no longer names the net of J3.100 (HDMI0_SCL)
- net HDMI0_SDA: no longer names the net of J3.99 (HDMI0_SDA)
- net HDMI1_CEC: no longer names the net of J3.49 (HDMI1_CEC)
- net HDMI1_CK_N: no longer names the net of J3.66 (HDMI1_CLK_N)
- net HDMI1_CK_P: no longer names the net of J3.64 (HDMI1_CLK_P)
- net HDMI1_D0_N: no longer names the net of J3.60 (HDMI1_TX0_N)
- net HDMI1_D0_P: no longer names the net of J3.58 (HDMI1_TX0_P)
- net HDMI1_D1_N: no longer names the net of J3.54 (HDMI1_TX1_N)
- net HDMI1_D1_P: no longer names the net of J3.52 (HDMI1_TX1_P)
- net HDMI1_D2_N: no longer names the net of J3.48 (HDMI1_TX2_N)
- net HDMI1_D2_P: no longer names the net of J3.46 (HDMI1_TX2_P)
- net HDMI1_HOTPLUG: no longer names the net of J3.43 (HDMI1_HOTPLUG)
- net HDMI1_SCL: no longer names the net of J3.47 (HDMI1_SCL)
- net HDMI1_SDA: no longer names the net of J3.45 (HDMI1_SDA)
- net USB3-0-D_N: no longer names the net of J3.36 (USB3-0-D_N)
- net USB3-0-D_P: no longer names the net of J3.34 (USB3-0-D_P)
- net USB3-0-RX_N: no longer names the net of J3.28 (USB3-0-RX_N)
- net USB3-0-RX_P: no longer names the net of J3.30 (USB3-0-RX_P)
- net USB3-0-TX_N: no longer names the net of J3.40 (USB3-0-TX_N)
- net USB3-0-TX_P: no longer names the net of J3.42 (USB3-0-TX_P)
- net USB3-1-D_N: no longer names the net of J3.65 (USB3-1-D_N)
- net USB3-1-D_P: no longer names the net of J3.63 (USB3-1-D_P)
- net USB3-1-RX_N: no longer names the net of J3.57 (USB3-1-RX_N)
- net USB3-1-RX_P: no longer names the net of J3.59 (USB3-1-RX_P)
- net USB3-1-TX_N: no longer names the net of J3.69 (USB3-1-TX_N)
- net USB3-1-TX_P: no longer names the net of J3.71 (USB3-1-TX_P)
- net USBOTG_ID: no longer names the net of J3.1 (USB_OTG_ID)
- net VBUS_EN: no longer names the net of J3.11 (VBUS_EN)
- no-connect marks 1 -> 43
