File: v3/CM5IO.kicad_sch (KiCad schematic)
At the start: 9 parts, among them J1 TYPE-C-31-M-12

Commit message: adding power management to board
Parts:
- added R8: 10k, Resistor_SMD:R_0402_1005Metric, symbol Device:R
- added U1: TS3USB221ARSER, footprint:UQFN-10_L2.0-W1.5-P0.50-BL, symbol TS3USB221ARSER:TS3USB221ARSER
Connections:
- net +3.3v: now also R8.1, U1.10 (VCC)
- net GND: now also U1.5 (GND), U1.6 (OE#)
- net USB2_N: now also U1.7 (D-)
- net USB2_P: now also U1.8 (D+)
- new net CM5_USB2_N: U1.4 (2D-)
- new net CM5_USB2_P: U1.3 (2D+)
- new net DSEL: R8.2, U1.9 (S)
- new net PWR_D+: U1.1 (1D+)
- new net PWR_D-: U1.2 (1D-)
Other:
- added sheet Power (power.kicad_sch)
- sheet CM5_GPIO ( Ethernet, GPIO, SDCARD) ports: added PWR_BUT, PWR_SCL, PWR_SDA; removed none

Commit message: Finalise v1.0 design
Parts:
- removed C1, C2: 100n, Capacitor_SMD:C_0402_1005Metric, symbol Device:C
- removed R1: 2.2K 1%, Resistor_SMD:R_0402_1005Metric, symbol Device:R
- U1: renamed from U6; now not fitted
- U2: renamed from U1; LCSC C128396 -> (none); LCSC PN (none) -> C128396
- renumbered R8 to R1
Connections:
- net +5v renamed Vbus
Other:
- sheet CM5_GPIO ( Ethernet, GPIO, SDCARD) ports: added none; removed CC1, CC2, GPIO_VREF, USBOTG
- sheet CM5_HighSpeed ports: added none; removed +5v, GPIO_VREF, USBOTG_ID
- sheet Power ports: added CC1, CC2, PMID; removed +5V
- note removed: "Discharge Resistor Needed by some Type C PSUs"

Commit message: updated hardware files
Changed lines of the file:
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@@
 	)
 	(label "PWR_SCL"
-		(at 203.2 44.45 0)
+		(at 203.2 46.99 0)
 		(effects
 			(font
@@
 	)
 	(label "PWR_SDA"
-		(at 203.2 46.99 0)
-		(effects
-			(font
+		(at 203.2 44.45 0)
+		(effects
+			(font
