File: v3/power.kicad_sch (KiCad schematic)
At the start: 24 parts, among them SW1 Right angle Tact button, U7 BQ25895RTW, U8 SN74LVC1G57DBVR

Commit message: Finalise v1.0 design
Parts:
- removed D4: LED, LED_SMD:LED_0603_1608Metric, symbol Device:LED
- removed L1: 2.2uH, Inductor_SMD:L_Vishay_IHLP-2020, symbol Device:L
- removed SW1: Right angle Tact button, Button_Switch_THT:SW_Tactile_SPST_Angled_PTS645Vx58-2LFS, symbol Switch:SW_Push
- added C10: 470nF, Capacitor_SMD:C_0402_1005Metric, symbol Device:C
- added C11: 1uF, Capacitor_SMD:C_0603_1608Metric, symbol Device:C
- added C9: 100nF, Capacitor_SMD:C_0402_1005Metric, symbol Device:C
- added J2: Conn_01x06_Pin, Connector_PinHeader_2.54mm:PinHeader_1x06_P2.54mm_Vertical, symbol Connector:Conn_01x06_Pin
- added J4: Conn_01x04_Pin, Connector_PinHeader_2.54mm:PinHeader_1x04_P2.54mm_Vertical, symbol Connector:Conn_01x04_Pin
- added L1: MHCI05018-1R0M-R8A, footprint:IND-SMD_L5.7-W5.4, symbol MHCI05018-1R0M-R8A:MHCI05018-1R0M-R8A
- added LED3: MHS171UBCT, footprint:LED-SMD_L2.1-W1.0-R-RD, symbol MHS171UBCT:MHS171UBCT
- added R13: 300k, Resistor_SMD:R_0402_1005Metric, symbol Device:R
- added R14: 200k, Resistor_SMD:R_0402_1005Metric, symbol Device:R
- added R15: 10k, Resistor_SMD:R_0402_1005Metric, symbol Device:R
- added R16: 1k, Resistor_SMD:R_0402_1005Metric, symbol Device:R
- added R17: 10mOhm, Resistor_SMD:R_2512_6332Metric, symbol Device:R
- added R18, R19: 5.1k, Resistor_SMD:R_0402_1005Metric, symbol Device:R
- added SW2: TS-1093C-A5B3-D1, footprint:SW-TH_TS-1093C-A5B3-D1, symbol TS-1093C-A5B3-D1:TS-1093C-A5B3-D1
- added U7: MAX17261xxTD, Package_DFN_QFN:TDFN-14-1EP_3x3mm_P0.4mm_EP1.78x2.35mm, symbol Battery_Management:MAX17261xxTD
- added U8: CH221K, footprint:SOT-23-6_L2.9-W1.6-P0.95-LS2.8-BL-2, symbol CH221K:CH221K
- R8: renamed from R12; value 260 -> 261; LCSC PN C25744 -> C25097
- renumbered C18 to C2, C17 to C3, C14 to C4, C12 to C5, C16 to C6, C15 to C7, C13 to C8, R14 to R12, R13 to R9, U7 to U5, U8 to U6
Connections:
- net +3.3v: now also J4.1 (Pin_1)
- net +BATT: now also C9.1, J2.2 (Pin_2), R13.1, U7.1 (TH), U7.6 (BATT)
- net GND: now also C11.2, J2.6 (Pin_6), J4.4 (Pin_4), R17.1, R18.1, R19.2, SW2.1, U7.7 (CSN), U8.2 (GND); no longer B1.2, B2.2
- net OTG: now also J2.3 (Pin_3)
- net PWR_CTRL: now also J2.1 (Pin_1), SW2.2
- net PWR_SCL: now also J4.3 (Pin_3), U7.14 (SCL)
- net PWR_SDA: now also J4.2 (Pin_2), U7.13 (SDA)
- net STAT: now also LED3.2 (K)
- net Vbus: now also J2.4 (Pin_4), R16.1
- net Vsys: now also L1.2
- net SW: now reaches C5.1, D3.2 (A), U5.19 (SW), U5.20 (SW)
- net SW: now also L1.1
- net at R9.2: now also LED3.1 (A)
- net +5V renamed PMID
- net PMID: now also J2.5 (Pin_5)
- new net: C11.1, R15.1, R16.2, U8.1 (VDD)
- new net: R15.2, U8.6 (CFG)
- new net: R13.2, R14.1, U7.10 (CELLX)
- new net: C10.1, U7.11 (REG)
- new net -BATT: B1.2, B2.2, C10.2, C9.2, R14.2, R17.2, U7.12 (ALRT), U7.15 (GND), U7.8 (GND), U7.9 (CSPL)
- new net CC1: R19.1, U8.4 (CC1)
- new net CC2: R18.2, U8.5 (CC2)
- no-connect marks 2 -> 6

Commit message: updated hardware files
Connections:
- net PWR_SCL: now also J4.2 (Pin_2); no longer J4.3 (Pin_3)
- net PWR_SDA: now also J4.3 (Pin_3); no longer J4.2 (Pin_2)
Changed lines of the file:
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@@
 	(hierarchical_label "PWR_SDA"
 		(shape bidirectional)
-		(at 144.78 175.26 0)
+		(at 144.78 177.8 0)
 		(effects
 			(font
@@
 	(hierarchical_label "PWR_SCL"
 		(shape bidirectional)
-		(at 144.78 177.8 0)
+		(at 144.78 175.26 0)
 		(effects
 			(font
